File: rail_splitter.kicad_sch (KiCad schematic)
At the start: 74 parts, among them J1 input +, J2 input -, J3 +load, J4 gnd load, J5 -load, J6 shunt+ display pos, J7 shunt- display pos, J8 shunt+ display neg, J9 shunt- display neg, Q1 PNP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

Commit message: pcb_v1
Parts:
- removed R25: 10k, Resistor_SMD:R_1206_3216Metric, symbol Device:R
- removed R28, R29: 1k, Resistor_SMD:R_1206_3216Metric, symbol Device:R
- removed U4: NE5532, Package_SO:SOIC-8_3.9x4.9mm_P1.27mm, symbol Amplifier_Operational:NE5532
- added Q8: NPN, Package_TO_SOT_SMD:SOT-23, symbol Simulation_SPICE:NPN
- added Q9: PNP, Package_TO_SOT_SMD:SOT-23, symbol Simulation_SPICE:PNP
- added R18: 1k, Resistor_SMD:R_1206_3216Metric, symbol Device:R
- RV2: value ~ -> RV2
- SW2: footprint (none) -> rail_lib:dpst
Connections:
- net CURR_LIMIT: now also U3.5 (+)
- net GND: no longer U3.5 (+)
- net INPUT+: now also Q9.3 (E)
- net INPUT-: now also Q8.3 (E)
- net at R26.2, U3.1: now also U3.6 (-); no longer R24.1
- net at R33.1: now also Q8.1 (C), Q9.1 (C)
- net at R24.2: now also D6.1 (K), R18.2; no longer U3.6 (-)
- net at U3.7: now also R27.2
- new net: Q8.2 (B), R24.1
- new net: Q9.2 (B), R18.1
Other:
- moved on the sheet: J5

Commit message: pcb verzija 3
Parts:
- removed SW2: SW_DPST, rail_lib:dpst, symbol Switch:SW_DPST
- added C3: 10n, Capacitor_SMD:C_1206_3216Metric, symbol Device:C
- added H1, H2, H3, H4: MountingHole, MountingHole:MountingHole_2.1mm, symbol Mechanical:MountingHole
- added SW3: SW_DPDT_x2, rail_lib:DPDT_bigger, symbol Switch:SW_DPDT_x2
- J1, J2, J3, J4, J5: footprint Connector:Banana_Jack_1Pin -> rail_lib:holder
- Q11, Q7: footprint Package_TO_SOT_THT:TO-220-3_Vertical -> Package_TO_SOT_SMD:SOT-23
- Q4: value dar -> N
- renumbered Qdar1 to P1
Connections:
- net INPUT+: now also C3.1, SW3.2 (B)
- net INPUT-: now also C3.2, SW3.5 (B)
- net enable -: now also SW3.6 (C)
- net enable+: now also SW3.3 (C)

Commit message: review, malo pomerano
Parts:
- added C10, C6, C7, C8, C9: 100n, Capacitor_SMD:C_1206_3216Metric, symbol Device:C
Connections:
- net GND: now also C6.2, C7.1, C8.2, C9.1
- net INPUT+: now also C10.1, C6.1, C8.1
- net INPUT-: now also C10.2, C7.2, C9.2
Other:
- moved on the sheet: U2C, U3C
