File: rail_splitter.kicad_sch (KiCad schematic)
At the start: 78 parts, among them J1 input +, J2 input -, J3 +load, J4 gnd load, J5 -load, J6 shunt+ display pos, J7 shunt- display pos, J8 shunt+ display neg, J9 shunt- display neg, P1 PNP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

Commit message: nova verzija pcb
Parts:
- removed D6: 1N4148WT, Diode_SMD:D_SOD-523, symbol Diode:1N4148WT
- added C10, C11, C12, C6, C7, C8, C9: 10n, Capacitor_SMD:C_1206_3216Metric, symbol Device:C
- added D7: LED, LED_THT:LED_D4.0mm, symbol Device:LED
- D4: footprint LED_SMD:LED_1206_3216Metric -> LED_THT:LED_D4.0mm
Connections:
- net GND: now also C3.2, C10.1, C11.1, C12.1, C6.2, C7.2, C8.2, C9.1
- net INPUT+: now also C6.1, C7.1, C8.1
- net INPUT-: now also C10.2, C11.2, C12.2, C9.2; no longer C3.2
- net at R18.2, R24.2: now also D7.1 (K)
- net at Q6.1 (C), R16.1, R17.2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: now also D7.2 (A)
Other:
- note added: "zamenio umesto obicne diode"
