File: rail_splitter.kicad_sch (KiCad schematic)
At the start: 85 parts, among them J1 input +, J2 input -, J3 +load, J4 gnd load, J5 -load, J6 shunt+ display pos, J7 shunt- display pos, J8 shunt+ display neg, J9 shunt- display neg, P1 PNP, Q1 PNP, Q11 NMOS, Q2 NPN, Q3 NPN, Q4 N, Q5 NPN, Q6 PNP, Q7 PMOS, Q8 NPN, Q9 PNP, SW1 SW_Push, SW3 SW_DPDT_x2, U1 OP07, U2 NE5532, U3 NE5532, U5 LM2936-3.3, U6 NE5532

Commit message: pcb izmene
Parts:
- J6, J8: footprint Connector_PinHeader_1.00mm:PinHeader_1x02_P1.00mm_Vertical -> Connector_PinHeader_2.54mm:PinHeader_1x01_P2.54mm_Vertical
- J7, J9: footprint Connector_PinHeader_1.00mm:PinHeader_1x01_P1.00mm_Vertical -> Connector_PinHeader_2.54mm:PinHeader_1x01_P2.54mm_Vertical
Changed lines of the file:
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@@
 			)
 		)
-		(property "Footprint" "Connector_PinHeader_1.00mm:PinHeader_1x02_P1.00mm_Vertical"
+		(property "Footprint" "Connector_PinHeader_2.54mm:PinHeader_1x01_P2.54mm_Vertical"
 			(at 220.98 182.88 0)
 			(effects
@@
 			)
 		)
-		(property "Footprint" "Connector_PinHeader_1.00mm:PinHeader_1x02_P1.00mm_Vertical"
+		(property "Footprint" "Connector_PinHeader_2.54mm:PinHeader_1x01_P2.54mm_Vertical"
 			(at 326.39 21.59 0)
 			(effects
@@
 			)
 		)
-		(property "Footprint" "Connector_PinHeader_1.00mm:PinHeader_1x01_P1.00mm_Vertical"
+		(property "Footprint" "Connector_PinHeader_2.54mm:PinHeader_1x01_P2.54mm_Vertical"
 			(at 215.9 158.75 0)
 			(effects
@@
 			)
 		)
-		(property "Footprint" "Connector_PinHeader_1.00mm:PinHeader_1x01_P1.00mm_Vertical"
+		(property "Footprint" "Connector_PinHeader_2.54mm:PinHeader_1x01_P2.54mm_Vertical"
 			(at 375.92 31.75 0)
 			(effects

Commit message: 67
Parts:
- added Q10: PMOS, Package_TO_SOT_SMD:SOT-23, symbol Simulation_SPICE:PMOS
- added Q12: NMOS, Package_TO_SOT_SMD:SOT-23, symbol Simulation_SPICE:NMOS
- C1, C10, C11, C12, C3, C6, C7, C8, C9: LCSC (none) -> C1846
- C2: value 0.22u -> 100n; LCSC (none) -> C1945
- C4: LCSC (none) -> C1945
- C5: LCSC (none) -> C1849
- D1, D2, D3, D5: footprint Diode_SMD:D_SOD-523 -> Diode_SMD:D_SOD-323; LCSC (none) -> C2128
- Q1, Q6, Q9: LCSC (none) -> C8326
- Q11: LCSC (none) -> C20917
- Q2, Q3, Q5, Q8: LCSC (none) -> C2145
- Q7: LCSC (none) -> C10487
- R10, R13, R14, R17, R18, R19, R21, R22, R24, R27, R33, R34, R35, R36, R37, R38, R6, R9: LCSC (none) -> C4410
- R11, R12, R15, R16, R23, R26: LCSC (none) -> C17902
- R3: value 67 -> 100; LCSC (none) -> C17901
- R4: value 5.6k -> 4.7K; LCSC (none) -> C17936
- R5: value 3.3k -> 4.7K; LCSC (none) -> C17936
- R7: value 470 -> 300; LCSC (none) -> C17887
- U2, U3, U6: LCSC (none) -> C7426
Connections:
- net INPUT+: now also Q10.3 (S)
- net INPUT-: now also Q12.3 (S)
- net enable -: now also Q12.2 (G)
- net enable+: now also Q10.2 (G)
- net at J8.1 (Pin_1), Q11.1 (D), R20.2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: now also Q12.1 (D)
- net at J6.1 (Pin_1), Q7.1 (D), R8.1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: now also Q10.1 (D)
Other:
- note removed: "zamenio umesto obicne diode"
- moved on the sheet: C4, C5, J6, R11, R33, R8, U5
