File: rail_splitter.kicad_sch (KiCad schematic)
At the start: 91 parts, among them J1 input +, J2 input -, J3 +load, J4 gnd load, J5 -load, J6 shunt+ display pos, J7 shunt- display pos, J8 shunt+ display neg, J9 shunt- display neg, P1 PNP, Q1 PNP, Q10 PMOS, Q11 NMOS, Q12 NMOS, Q2 NPN, Q3 NPN, Q4 N, Q5 NPN, Q6 PNP, Q7 PMOS, Q8 NPN, Q9 PNP, SW1 SW_Push, SW3 SW_DPDT_x2, U1 OP07, U2 NE5532, U3 NE5532, U5 LM2936-3.3, U6 NE5532

Commit message: overa nova
Parts:
- removed C40, C6, C7: 100n, Capacitor_SMD:C_1206_3216Metric, symbol Device:C
- renumbered C13 to C1, C9 to C10, C2 to C11, C5 to C12, C8 to C15, C10 to C16, C1 to C2, C46 to C3, C41 to C4, C3 to C5, C12 to C6, C4 to C8, C47 to C9, D2 to D1, D1 to D2, D4 to D3, D7 to D4, D3 to D5, D5 to D6, H4 to H1, H3 to H2, H2 to H3, H1 to H4, J2 to J1, J1 to J2, J4 to J3, J9 to J4, J8 to J5, J5 to J6, J6 to J7, J3 to J8, J7 to J9, Q3 to Q10, Q10 to Q11, Q7 to Q12, Q4 to Q3, Q9 to Q4, Q8 to Q5, Q11 to Q6, Q12 to Q7, Q6 to Q8, Q5 to Q9, R36 to R1, R38 to R10, R1 to R11, R2 to R12, R18 to R13, R24 to R14, R19 to R15, R33 to R16, R16 to R17, R15 to R18, R20 to R19, R34 to R2, R14 to R20, R22 to R21, R21 to R22, R26 to R24, R13 to R25, R12 to R26, R17 to R27, R11 to R28, R9 to R29, R35 to R3, R10 to R30, R27 to R31, R8 to R32, R37 to R4, R4 to R5, R3 to R6, R5 to R7, R6 to R8, R7 to R9, RV2 to RV1, RV1 to RV2, RV4 to RV3, RV3 to RV4, SW3 to SW1, SW1 to SW2, U6 to U2, U2 to U3, U5 to U4, U2 to U5, U3 to U5
Connections:
- net CURR_LIMIT: now also U3.5 (+), U5.6 (-); no longer U3.6 (-), U5.5 (+)
- net at R24.2, U3.1: now also U3.6 (-); no longer U5.6 (-)
- net at R26.2, U5.1: now also U5.5 (+); no longer U3.5 (+)
- net at R31.2: now also U3.7; no longer U5.7
- net at R25.1: now also U5.7; no longer U3.7
Other:
- note added: "Outpout enable /disable switch"
- note added: "Referentni napon"
- moved on the sheet: C10, C12, C15, C16, C8, C9, RV4, SW1A, SW1B, U3B, U3C, U4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

Commit message: cleared errors
Connections:
- net GNDD is gone; now on net GND: C12.2, C8.2, RV3.3, RV4.3, U4.2 (GND)

Commit message: rev
Parts:
- removed J4: shunt- display neg, Connector_PinHeader_2.54mm:PinHeader_1x01_P2.54mm_Vertical, symbol Connector:Conn_01x01_Socket
- removed J5: shunt+ display neg, Connector_PinHeader_2.54mm:PinHeader_1x01_P2.54mm_Vertical, symbol Connector:Conn_01x01_Socket
- removed J7: shunt+ display pos, Connector_PinHeader_2.54mm:PinHeader_1x01_P2.54mm_Vertical, symbol Connector:Conn_01x01_Socket
- removed J9: shunt- display pos, Connector_PinHeader_2.54mm:PinHeader_1x01_P2.54mm_Vertical, symbol Connector:Conn_01x01_Socket
- removed P1: PNP, Package_TO_SOT_THT:TO-220-3_Vertical, symbol Simulation_SPICE:PNP
- removed Q1, Q4, Q8: PNP, Package_TO_SOT_SMD:SOT-23, symbol Simulation_SPICE:PNP
- removed Q10, Q2, Q5, Q9: NPN, Package_TO_SOT_SMD:SOT-23, symbol Simulation_SPICE:NPN
- removed Q11, Q12: PMOS, Package_TO_SOT_SMD:SOT-23, symbol Simulation_SPICE:PMOS
- removed Q3: N, Package_TO_SOT_THT:TO-220-3_Vertical, symbol Simulation_SPICE:NPN
- removed Q6, Q7: NMOS, Package_TO_SOT_SMD:SOT-23, symbol Simulation_SPICE:NMOS
- removed R13, R14, R15: 1k, Resistor_SMD:R_1206_3216Metric, symbol Device:R
- added C17: 10n, Capacitor_SMD:C_1206_3216Metric, symbol Device:C
- added D7: 1N4148WT, Diode_SMD:D_SOD-323, symbol Diode:1N4148WT
- added Q11, Q12: AO3401A, Package_TO_SOT_SMD:SOT-23, symbol Transistor_FET:AO3401A
- added Q13: BD909, Package_TO_SOT_THT:TO-220-3_Vertical, symbol Transistor_BJT:BD909
- added Q14: BD910, Package_TO_SOT_THT:TO-220-3_Vertical, symbol Transistor_BJT:BD910
- added Q15, Q16, Q17, Q3, Q5: MMBT5551L, Package_TO_SOT_SMD:SOT-23, symbol Transistor_BJT:MMBT5551L
- added Q6, Q7: AO3400A, Package_TO_SOT_SMD:SOT-23, symbol Transistor_FET:AO3400A
- added Q8: MMBT5401, Package_TO_SOT_SMD:SOT-23, symbol Transistor_BJT:MMBTA92
Connections:
- net CURR_LIMIT: now also U5.2 (-); no longer U3.5 (+)
- net GND: now also C17.2, Q16.2 (E), Q17.2 (E)
- net INPUT+: now also R16.1, Q11.3 (D), Q12.3 (D), Q13.2 (C), Q8.2 (E)
- net INPUT-: now also R27.1, Q14.2 (C), Q5.2 (E), Q6.2 (S), Q7.2 (S)
- net enable -: now also SW1.4 (A), Q5.3 (C), Q6.1 (G), Q7.1 (G); no longer SW1.6 (C)
- net enable+: now also D4.2 (A), R27.2, Q11.1 (G), Q12.1 (G), Q8.3 (C); no longer R27.1
- net at R12.2: now also Q14.3 (E)
- net at R19.2: now also R21.2, Q6.3 (D), Q7.3 (D); no longer R22.2
- net at D5.1 (K), D6.1 (K): now also Q16.1 (B)
- net at R24.1, U3.2 (-): now also R21.1; no longer R21.2
- net at R24.2, U3.1: now also U5.3 (+); no longer U3.6 (-)
- net at C2.1, R7.1, U1.6: now also Q13.1 (B), Q15.3 (C), Q3.2 (E)
- net at R11.1: now also Q13.3 (E)
- net at R20.2: now also Q16.3 (C), Q17.3 (C)
- net at D4.1 (K): now also R17.1, D7.2 (A)
- net at R29.1, R32.1: now also Q11.2 (S), Q12.2 (S)
- net at C11.2, R18.2, R20.1: now also Q8.1 (B)
- net at D6.2 (A): now also R31.2; no longer R31.1
- net at R7.2, RV2.1: now also Q15.1 (B)
- net at R17.2, SW2.2: now also C17.1, Q17.1 (B)
- net at D2.1 (K), R5.1: now also Q3.1 (B)
- net at J6.1 (Pin_1), R19.1: now also R22.2; no longer R21.1
- net at R26.2, U5.5 (+): now also U3.7; no longer U5.1
- net at R26.1, R30.2: now also U3.6 (-); no longer U5.2 (-)
- net at R28.1, R29.2: now also U3.5 (+); no longer U5.3 (+)
- net at C2.2, R8.2, R9.1: now also Q14.1 (B), Q15.2 (E)
- net at R6.2: now also Q3.3 (C)
- new net: D7.1 (K), Q5.1 (B)
- new net: R31.1, U5.1
Other:
- note added: "Output enable /disable switch"
- note removed: "Outpout enable /disable switch"
- moved on the sheet: C10, C15, C16, C9, D5, D6, J1, J6, J8, R16, R17, R19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
