File: rail_splitter.kicad_pcb (KiCad board)
At the start: 2 copper layers, 100 x 100 mm, 74 parts, among them J1 input +, J2 input -, J3 +load, J4 gnd load, J5 -load, P1 PNP, Q1 PNP, Q11 NMOS, Q2 NPN, Q3 NPN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

Commit message: nova verzija pcb
Parts:
- removed D6: 1N4148WT, Diode_SMD:D_SOD-523
- added C10: 10n, Capacitor_SMD:C_1206_3216Metric, B.Cu at (127.2, 66.8)
- added C11: 10n, Capacitor_SMD:C_1206_3216Metric, B.Cu at (142.0, 138.2)
- added C12: 10n, Capacitor_SMD:C_1206_3216Metric, B.Cu at (108.2, 91.3)
- added C6: 10n, Capacitor_SMD:C_1206_3216Metric, B.Cu at (138.4, 127.6)
- added C7: 10n, Capacitor_SMD:C_1206_3216Metric, B.Cu at (68.7, 87.9)
- added C8: 10n, Capacitor_SMD:C_1206_3216Metric, B.Cu at (126.3, 78.8)
- added C9: 10n, Capacitor_SMD:C_1206_3216Metric, B.Cu at (71.5, 99.5)
- added D7: LED, LED_THT:LED_D4.0mm, F.Cu at (64.0, 129.8)
- added J6: shunt+ display pos, Connector_PinHeader_1.00mm:PinHeader_1x02_P1.00mm_Vertical, F.Cu at (66.0, 75.8)
- added J7: shunt- display pos, Connector_PinHeader_1.00mm:PinHeader_1x01_P1.00mm_Vertical, F.Cu at (65.2, 79.2)
- added J8: shunt+ display neg, Connector_PinHeader_1.00mm:PinHeader_1x02_P1.00mm_Vertical, F.Cu at (136.0, 83.2)
- added J9: shunt- display neg, Connector_PinHeader_1.00mm:PinHeader_1x01_P1.00mm_Vertical, F.Cu at (136.0, 87.5)
- C1, R1, R2: moved to B.Cu
- D4: footprint LED_SMD:LED_1206_3216Metric -> LED_THT:LED_D4.0mm
- moved R8 77.2 mm to (71.5, 82.2), turned to 180 degrees
- moved D3 75.6 mm to (60.4, 95.2)
- moved R13 75.2 mm to (62.0, 92.2), turned to 180 degrees
- moved R12 73.0 mm to (67.5, 97.9), turned to 180 degrees
- moved R20 69.8 mm to (123.3, 85.5), turned to 180 degrees
- moved D5 69.0 mm to (135.0, 71.9), turned to -90 degrees
- moved Q7 67.1 mm to (78.3, 82.2), turned to 0 degrees
- moved U2 66.8 mm to (68.5, 92.8), turned to 180 degrees
- moved R27 63.1 mm to (133.3, 75.0), turned to 180 degrees
- moved Q11 60.4 mm to (116.7, 86.0), turned to 180 degrees
- moved R10 60.0 mm to (75.2, 91.7), turned to 180 degrees
- moved R23 59.4 mm to (124.2, 69.5), turned to 0 degrees
- moved R9 57.2 mm to (75.2, 94.2), turned to 180 degrees
- moved R26 56.8 mm to (132.3, 70.7), turned to -90 degrees
- moved U3 56.4 mm to (126.7, 74.4), turned to 0 degrees
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Connections:
- C3 pad 2: INPUT- -> GND
Routing:
- net Net-(Q8-C): track 25.8 -> 177.8 mm, vias 0 -> 5
- net /GND_SET: track 32.3 -> 151.1 mm, vias 0 -> 3
- net INPUT-: track 240.1 -> 314.8 mm, vias 2 -> 5
- net enable+: track 128.4 -> 56.6 mm, vias 2 -> 4
- net Net-(J3-Pin_1): track 57.9 -> 113.9 mm, vias 2 -> 0
- net GND: track 17.6 -> 72.0 mm, vias 7 -> 15
- net Net-(J8-Pin_1): track 100.3 -> 50.5 mm
- net +3.3V: track 83.6 -> 40.8 mm, vias 0 -> 2
- net Net-(J5-Pin_1): track 66.5 -> 106.9 mm, vias 2 -> 0
- net Net-(D7-A): track 31.0 -> 70.9 mm, vias 0 -> 2
- net INPUT+: track 404.9 -> 368.8 mm, vias 5 -> 11
- net enable -: track 19.4 -> 52.3 mm, vias 1 -> 2
- net Net-(J6-Pin_1): track 42.5 -> 28.0 mm
- net CURR_LIMIT: track 141.2 -> 154.0 mm, vias 6 -> 5
- net Net-(D3-K): track 119.6 -> 130.0 mm, vias 4 -> 2
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