File: rail_splitter.kicad_pcb (KiCad board)
At the start: 2 copper layers, 100 x 100 mm, 85 parts, among them J1 input +, J2 input -, J3 +load, J4 gnd load, J5 -load, J6 shunt+ display pos, J7 shunt- display pos, J8 shunt+ display neg, J9 shunt- display neg, P1 PNP, Q1 PNP, Q11 NMOS, Q2 NPN, Q3 NPN, Q4 N, Q5 NPN, Q6 PNP, Q7 PMOS, Q8 NPN, Q9 PNP, SW1 SW_Push, SW3 SW_DPDT_x2, U1 OP07, U2 NE5532, U3 NE5532, U5 LM2936-3.3, U6 NE5532

Commit message: pcb izmene
Parts:
- J6, J8: footprint Connector_PinHeader_1.00mm:PinHeader_1x02_P1.00mm_Vertical -> Connector_PinHeader_2.54mm:PinHeader_1x01_P2.54mm_Vertical
- J7, J9: footprint Connector_PinHeader_1.00mm:PinHeader_1x01_P1.00mm_Vertical -> Connector_PinHeader_2.54mm:PinHeader_1x01_P2.54mm_Vertical
- moved J6 70.0 mm to (60.5, 145.5), turned to 0 degrees
- moved J7 66.0 mm to (67.8, 145.2), turned to 0 degrees
- moved J8 62.6 mm to (139.0, 145.8)
- moved J9 58.3 mm to (133.2, 145.8)
- moved R8 46.7 mm to (70.5, 129.0), turned to -90 degrees
- moved C10 24.9 mm to (142.0, 86.8), turned to 90 degrees
- moved D5 24.1 mm to (133.2, 96.0), turned to 0 degrees
- moved R26 21.9 mm to (138.1, 91.8), turned to 180 degrees
- moved R23 20.7 mm to (139.3, 83.8), turned to -90 degrees
- moved R21 18.2 mm to (136.5, 79.3), turned to 90 degrees
- moved R27 17.9 mm to (133.8, 92.8), turned to 90 degrees
- moved R3 14.9 mm to (107.0, 86.0)
- moved R22 14.6 mm to (133.8, 79.3), turned to -90 degrees
- moved R4 14.3 mm to (102.0, 85.5)
- moved U3 14.1 mm to (134.4, 86.3), turned to -90 degrees
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Routing:
- net GND: track 72.0 -> 236.2 mm, vias 15 -> 7
- net INPUT-: track 314.8 -> 452.7 mm, vias 5 -> 10
- net Net-(J8-Pin_1): track 50.5 -> 102.0 mm, vias 0 -> 1
- net Net-(J6-Pin_1): track 28.0 -> 76.0 mm, vias 0 -> 1
- net Net-(Q8-C): track 177.8 -> 134.3 mm, vias 5 -> 4
- net Net-(J3-Pin_1): track 113.9 -> 72.0 mm, vias 0 -> 2
- net Net-(U3A--): track 14.3 -> 39.6 mm
- net Net-(Q1-C): track 63.5 -> 40.4 mm, vias 2 -> 0
- net /GND_SET: track 151.1 -> 128.6 mm
- net Net-(J5-Pin_1): track 106.9 -> 129.1 mm, vias 0 -> 3
- net +3.3V: track 40.8 -> 56.9 mm, vias 2 -> 0
- net Net-(Q2-B): track 16.1 -> 30.0 mm, vias 0 -> 2
- net Net-(D7-A): track 70.9 -> 84.2 mm, vias 2 -> 0
- net Net-(P1-B): track 49.0 -> 61.4 mm, vias 0 -> 5
- net Net-(D3-K): track 130.0 -> 119.0 mm, vias 2 -> 3
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
Commit message: 67
Parts:
- added Q10: PMOS, Package_TO_SOT_SMD:SOT-23, B.Cu at (79.8, 83.2)
- added Q12: NMOS, Package_TO_SOT_SMD:SOT-23, B.Cu at (121.3, 86.0)
- C2: value 0.22u -> 100n
- D1, D2, D3, D5: footprint Diode_SMD:D_SOD-523 -> Diode_SMD:D_SOD-323
- R3: value 67 -> 100
- R4: value 5.6k -> 4.7K
- R5: value 3.3k -> 4.7K
- R7: value 470 -> 300
- moved R20 4.75 mm to (123.3, 80.8)
- moved R17 4.25 mm to (71.7, 78.0)
- moved Q7 3.44 mm to (75.0, 83.2), turned to 90 degrees
Routing:
- net Net-(J6-Pin_1): track 76.0 -> 81.2 mm
- net INPUT-: track 452.7 -> 457.3 mm
- net Net-(D7-A): track 84.2 -> 80.0 mm
- net INPUT+: track 377.6 -> 381.8 mm
- net Net-(J5-Pin_1): track 129.1 -> 125.1 mm
- net enable+: track 54.2 -> 57.2 mm, vias 2 -> 3
- net enable -: track 63.3 -> 66.1 mm
- net Net-(J8-Pin_1): track 102.0 -> 103.9 mm
