File: rail_splitter.kicad_pcb (KiCad board)
At the start: 2 copper layers, 100 x 86.5 mm, 88 parts, among them J1 input +, J2 input -, J3 +load, J4 gnd load, J5 -load, J6 shunt+ display pos, J7 shunt- display pos, J8 shunt+ display neg, J9 shunt- display neg, P1 PNP, Q1 PNP, Q10 PMOS, Q11 NMOS, Q12 NMOS, Q2 NPN, Q3 NPN, Q4 N, Q5 NPN, Q6 PNP, Q7 PMOS, Q8 NPN, Q9 PNP, SW1 SW_Push, SW3 SW_DPDT_x2, U1 OP07, U2 NE5532, U3 NE5532, U5 LM2936-3.3, U6 NE5532

Commit message: overa2
Parts:
- moved R19 2.17 mm to (64.5, 136.0)
- moved D7 2.17 mm to (62.0, 130.5)
- moved Q8 2.17 mm to (57.0, 135.3)
- moved R18 2.17 mm to (57.3, 128.0)
- moved R24 2.17 mm to (57.3, 131.8)
Routing:
- net GND: track 22.1 -> 3.93 mm, vias 25 -> 26
- net INPUT-: track 476.6 -> 466.5 mm
- net INPUT+: track 403.7 -> 395.4 mm, vias 11 -> 13
- net CURR_LIMIT: track 164.9 -> 171.8 mm, vias 4 -> 2
- net enable -: track 66.1 -> 61.1 mm
- net /GND_SET: track 128.6 -> 125.6 mm, vias 3 -> 2
- net Net-(J6-Pin_1): track 81.2 -> 78.5 mm, vias 1 -> 0
- net Net-(J5-Pin_1): track 123.3 -> 125.3 mm
- net +3.3V: track 56.9 -> 58.8 mm
- net Net-(Q8-C): track 137.7 -> 138.8 mm
- net Net-(D3-K): track 118.8 -> 117.9 mm
- net Net-(Q9-B): track 5.02 -> 5.58 mm
- net Net-(J8-Pin_1): vias 1 -> 3

Commit message: overa3
Parts:
- moved Q9 0.50 mm to (55.1, 122.0)
Routing:
- net Net-(J5-Pin_1): track 125.3 -> 133.5 mm, vias 3 -> 6
- net CURR_LIMIT: track 171.8 -> 165.5 mm
- net GND: track 3.93 -> 0.97 mm, vias 26 -> 37
- net INPUT-: track 466.5 -> 469.3 mm, vias 12 -> 16
- net Net-(Q8-C): track 138.8 -> 136.2 mm, vias 4 -> 8
- net INPUT+: track 395.4 -> 396.9 mm
- net Net-(Q1-C): track 40.4 -> 39.6 mm
- net Net-(Q2-B): track 29.8 -> 29.0 mm
- net Net-(D3-K): track 117.9 -> 118.6 mm
- net enable+: vias 3 -> 5
