File: _restore_backup_2026-10-01T14-07-06-546/rail_splitter.kicad_pcb (KiCad board)
At the start: 2 copper layers, 100 x 86.5 mm, 88 parts, among them J1 input +, J2 input -, J3 +load, J4 gnd load, J5 -load, J6 shunt+ display pos, J7 shunt- display pos, J8 shunt+ display neg, J9 shunt- display neg, P1 PNP, Q1 PNP, Q10 PMOS, Q11 NMOS, Q12 NMOS, Q2 NPN, Q3 NPN, Q4 N, Q5 NPN, Q6 PNP, Q7 PMOS, Q8 NPN, Q9 PNP, SW1 SW_Push, SW3 SW_DPDT_x2, U1 OP07, U2 NE5532, U3 NE5532, U5 LM2936-3.3, U6 NE5532

Commit message: overa
Parts:
- removed C13: 47u, Capacitor_SMD:C_1206_3216Metric
- moved H1 14.3 mm to (54.3, 54.7)
- moved H3 13.4 mm to (146.7, 55.6)
- moved D5 0.50 mm to (133.2, 96.0)
- moved D2 0.42 mm to (91.9, 74.0)
Routing:
- net GND: track 22.1 -> 236.2 mm, vias 25 -> 7
- net INPUT+: track 403.7 -> 381.8 mm, vias 11 -> 9
- net INPUT-: track 476.6 -> 457.3 mm, vias 12 -> 10
- net Net-(Q8-C): track 137.7 -> 134.3 mm
- net Net-(J5-Pin_1): track 123.3 -> 125.1 mm
- net Net-(U3A--): track 41.3 -> 39.6 mm
- net Net-(D5-A): track 2.40 -> 1.75 mm
- removed copper zone on B.Cu, net GND
Other:
- board size 100 x 86.5 mm -> 100 x 100 mm
