File: _restore_backup_2026-10-01T14-07-06-546/rail_splitter.kicad_sch (KiCad schematic)
At the start: 88 parts, among them J1 input +, J2 input -, J3 +load, J4 gnd load, J5 -load, J6 shunt+ display pos, J7 shunt- display pos, J8 shunt+ display neg, J9 shunt- display neg, P1 PNP, Q1 PNP, Q10 PMOS, Q11 NMOS, Q12 NMOS, Q2 NPN, Q3 NPN, Q4 N, Q5 NPN, Q6 PNP, Q7 PMOS, Q8 NPN, Q9 PNP, SW1 SW_Push, SW3 SW_DPDT_x2, U1 OP07, U2 NE5532, U3 NE5532, U5 LM2936-3.3, U6 NE5532

Commit message: overa
Parts:
- removed C13: 47u, Capacitor_SMD:C_1206_3216Metric, symbol Device:C
Other:
- moved on the sheet: C10, C7, C8, C9, J1, J2, RV2, U1, U2C, U3C
